File: Led Cube 8x8x8/Schematics/Main.brd (EAGLE design)
At the start: 100 x 80 mm, 20 parts, among them J1 ATX24RH, Q1 16, U1 ATMEGA328P-PU, X1 9090-4V

Commit message: Updates
Parts:
- LED1: device SparkFun-LED:FKIT-LED-1206 -> SparkFun-LED:LED-0603
- R1: device SparkFun-Resistors:AXIAL-0.8 -> resistor-power:RWM8X45
- moved R1 16.0 mm to (29.6, 6.35)
- moved X1 1.27 mm to (83.8, 67.3), turned to 0 degrees
- turned LED1 to 180 degrees
Connections:
- net GND: now also R1.2, X1.2; no longer R1.P$2, X1.3
- net N$2: now also R1.1; no longer R1.P$1
- net VCC: now also X1.1; no longer X1.4
Routing:
- net GND: track 365.3 -> 386.6 mm
- net VCC: track 298.3 -> 300.8 mm
- net N$2: track 70.8 -> 73.2 mm
- net N$3: track 6.20 -> 6.74 mm
Other:
- board text added: "Main Board"
