File: Led Cube 8x8x8/Schematics/Main.sch (EAGLE design)
At the start: 13 parts, among them J1 ATX24RH, Q1 16, U1 ATMEGA328P-PU

Commit message: Added Missing Files
Parts:
- removed C1: 0.1uF, SparkFun-Capacitors:0.1UF-25V-5%(0603)
- added JP2: (no value), SparkFun-Connectors:M03X22X3_SILK_SM
- added JP3, JP4, JP5, JP6: M02LOCK, SparkFun-Connectors:M02LOCK
- added X1: 9090-4V, con-thomas-betts:9090-4V
- C2, C3: device SparkFun-Capacitors:0.1UF-25V-5%(0603) -> capacitor-wima:C2,5-3
Connections:
- removed net N$6: C1.2, U1.AREF
- new net N$13: JP2.3, U1.PB5
- new net N$14: JP2.5, U1.PB3
- new net N$16: JP2.6, U1.PB2
- new net N$17: JP2.4, U1.PB1
- new net N$18: JP2.2, U1.PD3
- net GND: now also JP3.1, JP4.1, JP5.1, JP6.1, X1.3; no longer C1.1
- net VCC: now also JP3.2, JP4.2, JP5.2, JP6.2, U1.AREF, X1.4
Other:
- moved on the sheet: C2, C3, Q1

Commit message: Files.
Parts:
- added C1, C5: (no value), SparkFun-Capacitors:CAP_POLPTH2
Connections:
- net GND: now also C1.-, C5.-
- net VCC: now also C1.+, C5.+
Changed lines of the file:
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@@
 <part name="GND8" library="SparkFun-Aesthetics" deviceset="GND" device=""/>
 <part name="GND9" library="SparkFun-Aesthetics" deviceset="GND" device=""/>
+<part name="C1" library="SparkFun-Capacitors" deviceset="CAP_POL" device="PTH2"/>
+<part name="C5" library="SparkFun-Capacitors" deviceset="CAP_POL" device="PTH2"/>
 </parts>
 <sheets>
@@
 <instance part="GND8" gate="1" x="-111.76" y="119.38" rot="R270"/>
 <instance part="GND9" gate="1" x="-111.76" y="104.14" rot="R270"/>
+<instance part="C1" gate="G$1" x="-180.34" y="167.64" rot="R180"/>
+<instance part="C5" gate="G$1" x="-116.84" y="134.62" rot="R180"/>
 </instances>
 <busses>
@@
 <pinref part="GND3" gate="1" pin="GND"/>
 <pinref part="JP1" gate="G$1" pin="6"/>
-<wire x1="-116.84" y1="172.72" x2="-200.66" y2="172.72" width="0.1524" layer="91"/>
+<wire x1="-116.84" y1="172.72" x2="-180.34" y2="172.72" width="0.1524" layer="91"/>
+<wire x1="-180.34" y1="172.72" x2="-200.66" y2="172.72" width="0.1524" layer="91"/>
 <wire x1="-200.66" y1="172.72" x2="-200.66" y2="162.56" width="0.1524" layer="91"/>
+<pinref part="C1" gate="G$1" pin="-"/>
+<junction x="-180.34" y="172.72"/>
 </segment>
 <segment>
@@
 <pinref part="GND5" gate="1" pin="GND"/>
 <wire x1="-109.22" y1="139.7" x2="-116.84" y2="139.7" width="0.1524" layer="91"/>
+<pinref part="C5" gate="G$1" pin="-"/>
+<junction x="-116.84" y="139.7"/>
 </segment>
 <segment>
@@
 <pinref part="U1" gate="A" pin="AREF"/>
 <wire x1="-172.72" y1="160.02" x2="-172.72" y2="154.94" width="0.1524" layer="91"/>
+<pinref part="C1" gate="G$1" pin="+"/>
+<wire x1="-172.72" y1="165.1" x2="-180.34" y2="165.1" width="0.1524" layer="91"/>
 </segment>
 <segment>
@@
 <pinref part="SUPPLY4" gate="G$1" pin="VCC"/>
 <wire x1="-111.76" y1="137.16" x2="-111.76" y2="132.08" width="0.1524" layer="91"/>
-</segment>
-<segment>
+<pinref part="C5" gate="G$1" pin="+"/>
+<wire x1="-116.84" y1="132.08" x2="-111.76" y2="132.08" width="0.1524" layer="91"/>
+</segment>
+<segment>

Commit message: Updates
Parts:
- LED1: device SparkFun-LED:LED-FKIT-1206 -> SparkFun-LED:LED0603
- R1: device SparkFun-Resistors:RESISTORPTH-2W -> resistor-power:RRWM8X45
Connections:
- net GND: now also X1.2; no longer X1.3
- net VCC: now also X1.1; no longer X1.4
Changed lines of the file:
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@@
 <part name="J1" library="SparkFun-Connectors" deviceset="ATX24" device="RH"/>
 <part name="U1" library="Atmel_By_element14_Batch_1-00" deviceset="ATMEGA328P-PU" device=""/>
-<part name="R1" library="SparkFun-Resistors" deviceset="RESISTOR" device="PTH-2W" value="22 O 10 W"/>
-<part name="LED1" library="SparkFun-LED" deviceset="LED" device="-FKIT-1206"/>
+<part name="R1" library="resistor-power" deviceset="R" device="RWM8X45" value="22 O 10 W"/>
+<part name="LED1" library="SparkFun-LED" deviceset="LED" device="0603"/>
 <part name="R2" library="resistor" deviceset="R-US_" device="M3216" value="422 Ohm 1/4W"/>
 <part name="GND1" library="SparkFun-Aesthetics" deviceset="GND" device=""/>
@@
 </segment>
 <segment>
-<pinref part="X1" gate="G$1" pin="3"/>
 <pinref part="GND5" gate="1" pin="GND"/>
-<wire x1="-109.22" y1="139.7" x2="-116.84" y2="139.7" width="0.1524" layer="91"/>
 <pinref part="C5" gate="G$1" pin="-"/>
-<junction x="-116.84" y="139.7"/>
+<pinref part="X1" gate="G$1" pin="2"/>
+<wire x1="-109.22" y1="142.24" x2="-116.84" y2="142.24" width="0.1524" layer="91"/>
+<wire x1="-116.84" y1="142.24" x2="-116.84" y2="139.7" width="0.1524" layer="91"/>
 </segment>
 <segment>
@@
 </segment>
 <segment>
-<pinref part="X1" gate="G$1" pin="4"/>
-<wire x1="-109.22" y1="137.16" x2="-111.76" y2="137.16" width="0.1524" layer="91"/>
 <pinref part="SUPPLY4" gate="G$1" pin="VCC"/>
-<wire x1="-111.76" y1="137.16" x2="-111.76" y2="132.08" width="0.1524" layer="91"/>
 <pinref part="C5" gate="G$1" pin="+"/>
 <wire x1="-116.84" y1="132.08" x2="-111.76" y2="132.08" width="0.1524" layer="91"/>
-</segment>
-<segment>
+<wire x1="-116.84" y1="132.08" x2="-124.46" y2="132.08" width="0.1524" layer="91"/>
+<wire x1="-124.46" y1="132.08" x2="-124.46" y2="144.78" width="0.1524" layer="91"/>
+<pinref part="X1" gate="G$1" pin="1"/>
+<wire x1="-124.46" y1="144.78" x2="-109.22" y2="144.78" width="0.1524" layer="91"/>
+</segment>
+<segment>
