File: WarpCore/Board/WarpCoreControl.brd (EAGLE design)
At the start: 100 x 80 mm, 15 parts

Commit message: Updates
Other:
- board size 100 x 80 mm -> 91.1 x 47 mm
Changed lines of the file:
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@@
 <board>
 <plain>
-<wire x1="0" y1="0" x2="100" y2="0" width="0" layer="20"/>
-<wire x1="100" y1="0" x2="100" y2="80" width="0" layer="20"/>
-<wire x1="100" y1="80" x2="0" y2="80" width="0" layer="20"/>
-<wire x1="0" y1="80" x2="0" y2="0" width="0" layer="20"/>
+<wire x1="0" y1="33.02" x2="91.11" y2="33.02" width="0" layer="20"/>
+<wire x1="91.11" y1="33.02" x2="91.11" y2="80" width="0" layer="20"/>
+<wire x1="91.11" y1="80" x2="0" y2="80" width="0" layer="20"/>
+<wire x1="0" y1="80" x2="0" y2="33.02" width="0" layer="20"/>
 </plain>
 <attributes>
