File: Cluster/Power/Power.brd (EAGLE design)
At the start: 83.5 x 47 mm, 20 parts, among them X1 KUSBVX, X2 KUSBVX, X3 KUSBVX, X4 KUSBVX, X5 KUSBVX, X6 KUSBVX, X7 KUSBVX, X8 KUSBVX

Commit message: updates
Parts:
- C1, C2, C3, C4, C5, C6, C7, C8: value 10uF -> 100uF; device SparkFun-Capacitors:CPOL-RADIAL-2.5MM-5MM -> SparkFun-Capacitors:CPOL-RADIAL-2.5MM-6.5MM
- moved C2 35.1 mm to (15.2, 62.2), turned to 0 degrees
- moved C7 33.0 mm to (63.5, 62.2)
- moved C6 19.4 mm to (49.5, 53.3), turned to 180 degrees
- moved C5 18.2 mm to (47.0, 62.2), turned to 0 degrees
- moved C4 17.8 mm to (30.5, 62.2)
- moved C8 17.3 mm to (62.2, 53.3), turned to 180 degrees
- moved C3 15.3 mm to (30.5, 53.3)
- moved C1 15.3 mm to (16.5, 53.3)
- moved X5 2.54 mm to (14.0, 47.0)
- moved X6 2.54 mm to (31.8, 47.0)
- moved X7 2.54 mm to (49.5, 47.0)
- moved X8 2.54 mm to (67.3, 47.0)
Routing:
- net GND: track 344.9 -> 373.4 mm
- net VCC: track 171.5 -> 198.0 mm
Other:
- board size 83.5 x 47 mm -> 86 x 47 mm
