File: Cluster/Power/Power.sch (EAGLE design)
At the start: 20 parts, among them X1 KUSBVX, X2 KUSBVX, X3 KUSBVX, X4 KUSBVX, X5 KUSBVX, X6 KUSBVX, X7 KUSBVX, X8 KUSBVX

Commit message: updates
Parts:
- C1, C2, C3, C4, C5, C6, C7, C8: value 10uF -> 100uF; device SparkFun-Capacitors:10UF-POLAR-RADIAL-2.5MM-25V-20% -> SparkFun-Capacitors:100UF-POLAR-RADIAL-2.5MM-25V-20%
Other:
- moved on the sheet: C2, C5, C6, C7, C8
